Commit message: Update : sensors all added

File: fusionbot_description/urdf/fusionbot.urdf (robot description, URDF)
Before this commit: robot fusionbot, 5 links, 4 joints
Links:
- added link camera_link, mass 0.01
- added link imu_link, mass 0.01
Joints:
- added joint camera_joint: type fixed, parent base_link, child camera_link, origin xyz=0.1 0.0 0.05 rpy=0 0 0, axis 0.0 0.0 0.0
- added joint imu_joint: type fixed, parent base_link, child imu_link, origin xyz=0.0 0.0 0.05 rpy=0 0 0, axis 0.0 0.0 0.0

File: fusionbot_description/urdf/fusionbot.urdf.xacro (robot description, xacro)
@@ -84,4 +84,16 @@
     </collision>
   </link>
+  <link name="imu_link">
+    <inertial>
+      <mass value="0.01"/>
+      <inertia ixx="1.0" ixy="0" ixz="0" iyy="1.0" iyz="0" izz="1.0"/>
+    </inertial>
+  </link>
+  <link name="camera_link">
+    <inertial>
+      <mass value="0.01"/>
+      <inertia ixx="1.0" ixy="0" ixz="0" iyy="1.0" iyz="0" izz="1.0"/>
+    </inertial>
+  </link>
   <joint name='base_link_joint' type='fixed'>
     <origin rpy="0 0 0" xyz="0 0 0" />
@@ -101,4 +113,16 @@
     <axis xyz="0.0 1.0 0.0" />
   </joint>
+  <joint name="imu_joint" type="fixed">
+    <origin rpy="0 0 0" xyz="0.0 0.0 0.05" />
+    <parent link="base_link" />
+    <child link="imu_link" />
+    <axis xyz="0.0 0.0 0.0" />
+  </joint>
+  <joint name="camera_joint" type="fixed">
+    <origin rpy="0 0 0" xyz="0.1 0.0 0.05" />
+    <parent link="base_link" />
+    <child link="camera_link" />
+    <axis xyz="0.0 0.0 0.0" />
+  </joint>
   <joint name="lidar_joint" type="fixed">
     <origin rpy="0 0 0" xyz="0.05 0.0 0.11" />

File: fusionbot_description/urdf/fusionbot_description.urdf (robot description, URDF)
Before this commit: robot fusionbot, 5 links, 4 joints
Links:
- added link camera_link, mass 0.01
- added link imu_link, mass 0.01
Joints:
- added joint camera_joint: type fixed, parent base_link, child camera_link, origin xyz=0.1 0.0 0.05 rpy=0 0 0, axis 0.0 0.0 0.0
- added joint imu_joint: type fixed, parent base_link, child imu_link, origin xyz=0.0 0.0 0.05 rpy=0 0 0, axis 0.0 0.0 0.0
