Commit message: Fix : sensor link inertia

File: fusionbot_description/urdf/fusionbot.urdf.xacro (robot description, xacro)
@@ -87,5 +87,5 @@
     <inertial>
       <mass value="0.01"/>
-      <inertia ixx="1.0" ixy="0" ixz="0" iyy="1.0" iyz="0" izz="1.0"/>
+      <inertia ixx="0.01" ixy="0" ixz="0" iyy="0.01" iyz="0" izz="0.01"/>
     </inertial>
   </link>
@@ -93,5 +93,5 @@
     <inertial>
       <mass value="0.01"/>
-      <inertia ixx="1.0" ixy="0" ixz="0" iyy="1.0" iyz="0" izz="1.0"/>
+      <inertia ixx="0.01" ixy="0" ixz="0" iyy="0.01" iyz="0" izz="0.01"/>
     </inertial>
   </link>
