Commit message: Desc editted

File: src_description/urdf/src_body.urdf (robot description, URDF)
Before this commit: robot src_body, 10 links, 9 joints
Links:
- link base_link: geometry collision mesh filename=package://src_description/meshes/base_link.stl scale=0.001 0.001 0.001; visual mesh filename=package://src_description/meshes/base_link.stl scale=0.001 0.001 0.001
- link lf_wheel_link: geometry collision mesh filename=package://src_description/meshes/wheel.stl scale=0.001 0.001 0.001; visual mesh filename=package://src_description/meshes/wheel.stl scale=0.001 0.001 0.001
- link logi_camera_link: geometry collision mesh filename=package://src_description/meshes/logi_camera.stl scale=0.001 0.001 0.001; visual mesh filename=package://src_description/meshes/logi_camera.stl scale=0.001 0.001 0.001
- link lr_wheel_link: geometry collision mesh filename=package://src_description/meshes/wheel.stl scale=0.001 0.001 0.001; visual mesh filename=package://src_description/meshes/wheel.stl scale=0.001 0.001 0.001
- link rf_wheel_link: geometry collision mesh filename=package://src_description/meshes/wheel.stl scale=0.001 0.001 0.001; visual mesh filename=package://src_description/meshes/wheel.stl scale=0.001 0.001 0.001
- link rplidar_a2_link: geometry collision mesh filename=package://src_description/meshes/rplidar_a2.stl scale=0.001 0.001 0.001; visual mesh filename=package://src_description/meshes/rplidar_a2.stl scale=0.001 0.001 0.001
- link rr_wheel_link: geometry collision mesh filename=package://src_description/meshes/wheel.stl scale=0.001 0.001 0.001; visual mesh filename=package://src_description/meshes/wheel.stl scale=0.001 0.001 0.001
