Commit message: racecourse done!!

File: src_gazebo/urdf/src_body.urdf (robot description, URDF)
Before this commit: robot src_body, 10 links, 9 joints
Links:
- link base_link: geometry collision mesh filename=/home/kimsooyoung/djhrd_ws/install/src_gazebo/share/src_gaz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 scale=0.001 0.001 0.001; visual mesh filename=/home/kimsooyoung/djhrd_ws/install/src_gazebo/share/src_gaz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 scale=0.001 0.001 0.001
- link lf_wheel_link: geometry collision mesh filename=/home/kimsooyoung/djhrd_ws/install/src_gazebo/share/src_gaz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 scale=0.001 0.001 0.001; visual mesh filename=/home/kimsooyoung/djhrd_ws/install/src_gazebo/share/src_gaz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 scale=0.001 0.001 0.001
- link logi_camera_link: geometry collision mesh filename=/home/kimsooyoung/djhrd_ws/install/src_gazebo/share/src_gaz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 scale=0.001 0.001 0.001; visual mesh filename=/home/kimsooyoung/djhrd_ws/install/src_gazebo/share/src_gaz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 scale=0.001 0.001 0.001
- link lr_wheel_link: geometry collision mesh filename=/home/kimsooyoung/djhrd_ws/install/src_gazebo/share/src_gaz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 scale=0.001 0.001 0.001; visual mesh filename=/home/kimsooyoung/djhrd_ws/install/src_gazebo/share/src_gaz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 scale=0.001 0.001 0.001
- link rf_wheel_link: geometry collision mesh filename=/home/kimsooyoung/djhrd_ws/install/src_gazebo/share/src_gaz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 scale=0.001 0.001 0.001; visual mesh filename=/home/kimsooyoung/djhrd_ws/install/src_gazebo/share/src_gaz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 scale=0.001 0.001 0.001
- link rplidar_a2_link: geometry collision mesh filename=/home/kimsooyoung/djhrd_ws/install/src_gazebo/share/src_gaz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 scale=0.001 0.001 0.001; visual mesh filename=/home/kimsooyoung/djhrd_ws/install/src_gazebo/share/src_gaz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 scale=0.001 0.001 0.001
- link rr_wheel_link: geometry collision mesh filename=/home/kimsooyoung/djhrd_ws/install/src_gazebo/share/src_gaz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 scale=0.001 0.001 0.001; visual mesh filename=/home/kimsooyoung/djhrd_ws/install/src_gazebo/share/src_gaz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 scale=0.001 0.001 0.001

File: src_gazebo/urdf/src_body.urdf.xacro (robot description, xacro)
@@ -3,6 +3,6 @@
   <xacro:include filename="$(find src_gazebo)/urdf/materials.xacro" />
   <xacro:include filename="$(find src_gazebo)/urdf/macros.xacro" />
+  <xacro:include filename="$(find src_gazebo)/urdf/src_body.gazebo" />
   <!-- <xacro:include filename="$(find src_gazebo)/urdf/src_body.trans" /> -->
-  <!-- <xacro:include filename="$(find src_gazebo)/urdf/src_body.gazebo" /> -->
   <link name="base_link">
     <inertial>
@@ -14,5 +14,5 @@
       <origin xyz="0 0 0" rpy="0 0 0"/>
       <geometry>
-        <mesh filename="package://src_gazebo/meshes/base_link.stl" scale="0.001 0.001 0.001"/>
+        <mesh filename="$(find src_gazebo)/meshes/base_link.stl" scale="0.001 0.001 0.001"/>
       </geometry>
       <material name="silver"/>
@@ -21,5 +21,5 @@
       <origin xyz="0 0 0" rpy="0 0 0"/>
       <geometry>
-        <mesh filename="package://src_gazebo/meshes/base_link.stl" scale="0.001 0.001 0.001"/>
+        <mesh filename="$(find src_gazebo)/meshes/base_link.stl" scale="0.001 0.001 0.001"/>
       </geometry>
     </collision>
@@ -49,12 +49,12 @@
       <origin xyz="0 0 0" rpy="0 0 0"/>
       <geometry>
-        <mesh filename="package://src_gazebo/meshes/wheel.stl" scale="0.001 0.001 0.001"/>
-      </geometry>
-      <material name="black"/>
-    </visual>
-    <collision>
-      <origin xyz="0 0 0" rpy="0 0 0"/>
-      <geometry>
-        <mesh filename="package://src_gazebo/meshes/wheel.stl" scale="0.001 0.001 0.001"/>
+        <mesh filename="$(find src_gazebo)/meshes/wheel.stl" scale="0.001 0.001 0.001"/>
+      </geometry>
+      <material name="black"/>
+    </visual>
+    <collision>
+      <origin xyz="0 0 0" rpy="0 0 0"/>
+      <geometry>
+        <mesh filename="$(find src_gazebo)/meshes/wheel.stl" scale="0.001 0.001 0.001"/>
       </geometry>
     </collision>
@@ -91,12 +91,12 @@
       <origin xyz="0 0 0" rpy="0 0 0"/>
       <geometry>
-        <mesh filename="package://src_gazebo/meshes/wheel.stl" scale="0.001 0.001 0.001"/>
-      </geometry>
-      <material name="black"/>
-    </visual>
-    <collision>
-      <origin xyz="0 0 0" rpy="0 0 0"/>
-      <geometry>
-        <mesh filename="package://src_gazebo/meshes/wheel.stl" scale="0.001 0.001 0.001"/>
+        <mesh filename="$(find src_gazebo)/meshes/wheel.stl" scale="0.001 0.001 0.001"/>
+      </geometry>
+      <material name="black"/>
+    </visual>
+    <collision>
+      <origin xyz="0 0 0" rpy="0 0 0"/>
+      <geometry>
+        <mesh filename="$(find src_gazebo)/meshes/wheel.stl" scale="0.001 0.001 0.001"/>
       </geometry>
     </collision>
@@ -118,12 +118,12 @@
       <origin xyz="0 0 0" rpy="0 0 0"/>
       <geometry>
-        <mesh filename="package://src_gazebo/meshes/wheel.stl" scale="0.001 0.001 0.001"/>
-      </geometry>
-      <material name="black"/>
-    </visual>
-    <collision>
-      <origin xyz="0 0 0" rpy="0 0 0"/>
-      <geometry>
-        <mesh filename="package://src_gazebo/meshes/wheel.stl" scale="0.001 0.001 0.001"/>
+        <mesh filename="$(find src_gazebo)/meshes/wheel.stl" scale="0.001 0.001 0.001"/>
+      </geometry>
+      <material name="black"/>
+    </visual>
+    <collision>
+      <origin xyz="0 0 0" rpy="0 0 0"/>
+      <geometry>
+        <mesh filename="$(find src_gazebo)/meshes/wheel.stl" scale="0.001 0.001 0.001"/>
       </geometry>
     </collision>
@@ -144,12 +144,12 @@
       <origin xyz="0 0 0" rpy="0 0 0"/>
       <geometry>
-        <mesh filename="package://src_gazebo/meshes/wheel.stl" scale="0.001 0.001 0.001"/>
-      </geometry>
-      <material name="black"/>
-    </visual>
-    <collision>
-      <origin xyz="0 0 0" rpy="0 0 0"/>
-      <geometry>
-        <mesh filename="package://src_gazebo/meshes/wheel.stl" scale="0.001 0.001 0.001"/>
+        <mesh filename="$(find src_gazebo)/meshes/wheel.stl" scale="0.001 0.001 0.001"/>
+      </geometry>
+      <material name="black"/>
+    </visual>
+    <collision>
+      <origin xyz="0 0 0" rpy="0 0 0"/>
+      <geometry>
+        <mesh filename="$(find src_gazebo)/meshes/wheel.stl" scale="0.001 0.001 0.001"/>
       </geometry>
     </collision>
@@ -170,5 +170,5 @@
       <origin xyz="0 0 0" rpy="0 0 0"/>
       <geometry>
-        <mesh filename="package://src_gazebo/meshes/rplidar_a2.stl" scale="0.001 0.001 0.001"/>
+        <mesh filename="$(find src_gazebo)/meshes/rplidar_a2.stl" scale="0.001 0.001 0.001"/>
       </geometry>
       <material name="silver"/>
@@ -177,5 +177,5 @@
       <origin xyz="0 0 0" rpy="0 0 0"/>
       <geometry>
-        <mesh filename="package://src_gazebo/meshes/rplidar_a2.stl" scale="0.001 0.001 0.001"/>
+        <mesh filename="$(find src_gazebo)/meshes/rplidar_a2.stl" scale="0.001 0.001 0.001"/>
       </geometry>
     </collision>
@@ -195,5 +195,5 @@
       <origin xyz="0 0 0" rpy="0 0 0"/>
       <geometry>
-        <mesh filename="package://src_gazebo/meshes/logi_camera.stl" scale="0.001 0.001 0.001"/>
+        <mesh filename="$(find src_gazebo)/meshes/logi_camera.stl" scale="0.001 0.001 0.001"/>
       </geometry>
       <material name="silver"/>
@@ -202,5 +202,5 @@
       <origin xyz="0 0 0" rpy="0 0 0"/>
       <geometry>
-        <mesh filename="package://src_gazebo/meshes/logi_camera.stl" scale="0.001 0.001 0.001"/>
+        <mesh filename="$(find src_gazebo)/meshes/logi_camera.stl" scale="0.001 0.001 0.001"/>
       </geometry>
     </collision>
